File: spring_2026_ID/diagrams/jakarta/jakarta_system.kicad_sch (KiCad schematic)
At the start: 36 parts, among them J1 220V AC 50Hz, J2 Pi-EzConnect (Adafruit 2711), J3 IP68 RJ45, J4 IP68 RJ45, SW1 IP67 Momentary, U1 Witty Pi 5 HAT+, U2 Raspberry Pi 5 (4GB/8GB), U3 512GB M.2 SSD + USB, U4 Quectel EG25-G + PU201

Commit message: procurement updates
Parts:
- U4: value Quectel EG25-G + PU201 -> Quectel EG25-G + EXVIST Mini PCIe-USB
Changed lines of the file:
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@@
   ;; LTE MODEM SECTION
   ;; ============================================
-  ;; Quectel EG25-G Modem + PU201
+  ;; Quectel EG25-G Modem + EXVIST Mini PCIe-USB Adapter
   (symbol
     (lib_id "RF_Module:Modem")
@@
       (effects (font (size 1.27 1.27)))
     )
-    (property "Value" "Quectel EG25-G + PU201"
+    (property "Value" "Quectel EG25-G + EXVIST Mini PCIe-USB"
       (at 342.9 187.96 0)
       (effects (font (size 1.27 1.27)))
