File: spring_2026_ID/diagrams/sukabumi/sukabumi_system.kicad_sch (KiCad schematic)
At the start: 28 parts, among them J1 Pi-EzConnect (Adafruit 2711), J2 SMA Bulkhead, J3 SMA Bulkhead, J4 5.5x2.1mm Barrel-to-Screw, J5 Bulgin PX0840 IP67 USB, K1 Numato 1-Ch USB Relay, SW1 IP67 Momentary Pushbutton, U1 Witty Pi 5 HAT+, U2 Raspberry Pi 5 (4GB/8GB), U3 512GB M.2 SSD + USB Enclosure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

Commit message: updated circuit diagrams
Parts:
- removed F2: 3A Blade Fuse, symbol Device:Fuse
- removed H1: VA Imaging MVEC167 Aluminum, symbol Mechanical:Housing
- removed J4: 5.5x2.1mm Barrel-to-Screw, symbol Connector:Barrel_Jack
- removed J5: Bulgin PX0840 IP67 USB, symbol Connector:USB_A
- removed K1: Numato 1-Ch USB Relay, symbol Relay:Relay_SPDT
- removed LED1: Tendelux AI4 850nm IR, symbol Device:LED_IR
- added ANT3: Proxicast ANT-122-S02 MIMO Puck (IP67), symbol Device:Antenna
- added J4: IP68 RJ45 Waterproof Coupler, symbol Connector:RJ45
- added J5: Cat6 Outdoor Shielded Cable, symbol Connector:RJ45
- added U5: Planet IPOE-260-12V PoE Injector, symbol Connector:Conn_01x04
- CAM1: value ELP/SVPRO 8MP IMX179 NoIR -> ANNKE C1200 PoE Camera
- F1: value 10A Blade Fuse -> 5A Inline Blade Fuse
- J2, J3: value SMA Bulkhead -> SMA Bulkhead (M12)
- SENS1: value DFRobot SEN0575 -> Hydreon RG-15
- U2: value Raspberry Pi 5 (4GB/8GB) -> Raspberry Pi 5 (8GB)
- U3: value 512GB M.2 SSD + USB Enclosure -> Samsung FIT Plus 256GB USB
- renumbered LED2 to LED1, LED3 to LED2, LED4 to LED3
Other:
- note added: "CAMERA (EXTERNAL) ANNKE C1200 - Factory-sealed IP67 12MP, 134 deg FOV, built-in IR LEDs"
- note added: "GPIO PIN ASSIGNMENTS: GPIO14 - UART TX (to Hydreon RG-15 RX) GPIO15 - UART RX (from Hydreon RG-15 TX) GPIO17 - Green LED (System OK) GPIO22 - Red LED (Error) GPIO23 - Maintenance button input (internal pull-up) GPIO27 - Yellow LED (Working)"
- note added: "NOTES: 1. PoE injector powered via Witty Pi switched 12V rail - camera boots with Pi, sleeps with Pi 2. No heaters installed (Sukabumi tropical climate, solar power budget constraint) 3. Conformal coat (MG 422C silicone) on Pi, Witty Pi, Pi-EzConnect PCBs 4. Status LEDs: Green=OK, Yellow=Working, Red=Error (all via 330R series resistors) 5. Long press (3s) maintenance button (GPIO23) enters WiFi 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"
- note added: "POWER PATH: Battery 12V -> TB1 -> Witty Pi 5 (5-26V in) Witty Pi -> 5V USB-C -> Pi 5 Witty Pi -> Switched 12V -> F1 5A Fuse -> Planet IPOE-260 PoE Injector PoE Injector DATA port -> Pi 5 Ethernet (data only) PoE Injector DATA+POWER port -> Cat6 outdoor -> ANNKE C1200 (48V PoE) Pi 5 USB 2.0 -> Quectel EG25-G LTE Modem (bus-powered) Pi 5 USB 3.0 -> Samsung FIT Plus 256GB (bus-powered)"
- note added: "PoE CAMERA SYSTEM Planet IPOE-260-12V injector + ANNKE C1200 Camera power-cycled with Pi via Witty Pi switched 12V rail"
- note added: "SENSORS Hydreon RG-15 rain gauge on UART serial (GPIO14/15)"
- note removed: "CAMERA USB camera in Gore-vented aluminum housing"
- note removed: "GPIO PIN ASSIGNMENTS: GPIO4 - Witty Pi shutdown signal GPIO17 - Witty Pi wake signal / Green LED GPIO27 - Yellow LED GPIO22 - Red LED GPIO5 - Maintenance button input GPIO2 - I2C SDA (rain gauge) GPIO3 - I2C SCL (rain gauge)"
- note removed: "IR ILLUMINATION USB Relay controlled, photocell in light"
- note removed: "NOTES: 1. All GPIO via Pi-EzConnect screw terminals 2. Conformal coat (MG 422C) on Pi, Witty Pi, relay PCBs 3. IR relay controlled by systemd service on boot 4. Status LEDs: Green=OK, Yellow=Working, Red=Error 5. Long press (3s) maintenance button enters WiFi hotspot mode"
- note removed: "SENSORS Rain gauge on I2C bus"

Commit message: procurement updates
Parts:
- U4: value Quectel EG25-G + PU201 -> Quectel EG25-G + EXVIST Mini PCIe-USB
Changed lines of the file:
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@@
   ;; LTE MODEM SECTION
   ;; ============================================
-  ;; Quectel EG25-G Modem + PU201
+  ;; Quectel EG25-G Modem + EXVIST Mini PCIe-USB Adapter
   (symbol
     (lib_id "RF_Module:Modem")
@@
       (effects (font (size 1.27 1.27)))
     )
-    (property "Value" "Quectel EG25-G + PU201"
+    (property "Value" "Quectel EG25-G + EXVIST Mini PCIe-USB"
       (at 254 66.04 0)
       (effects (font (size 1.27 1.27)))
     )
-    (property "Description" "LTE Cat 4 modem with USB adapter, supports Indonesian carriers (Telkomsel)"
+    (property "Description" "LTE Cat 4 Mini PCIe modem with EXVIST P2U52V02USB adapter, supports Indonesian carriers (Telkomsel)"
       (at 254 68.58 0)
       (effects (font (size 1.0 1.0)) hide)
